Commit message: Update robot meshes and URDF files, Change sphear -> cylinder for roller collision

File: urdf/walkie/base/base.urdf.xacro (robot description, xacro)
@@ -1,38 +1,32 @@
 <?xml version="1.0"?>
 <robot xmlns:xacro="http://ros.org/wiki/xacro">
-  <xacro:include filename="$(find walkie_description)/urdf/walkie/base/base.gazebo.xacro" />
-  <xacro:include filename="$(find walkie_description)/urdf/inertial_macros.xacro" />
-  <xacro:property name="bass_thickness" value="0.008" />
-  <xacro:property name="base_radian" value="0.040" />
-  <xacro:property name="base_mass" value="20.2" />
+  <xacro:include filename="$(find walkie_description)/urdf/walkie/base/base.gazebo.xacro"/>
+  <xacro:include filename="$(find walkie_description)/urdf/inertial_macros.xacro"/>
+  <xacro:include filename="$(find walkie_description)/urdf/color.xacro"/>
+  <xacro:property name="bass_thickness" value="0.008"/>
+  <xacro:property name="base_radian" value="0.040"/>
+  <xacro:property name="base_mass" value="20.2"/>
   <xacro:macro name="base_v0" params="parent *joint_origin">
     <joint name="base_link_joint" type="fixed">
-      <xacro:insert_block name="joint_origin" />
-      <parent link="${parent}" />
-      <child link="base_link" />
+      <xacro:insert_block name="joint_origin"/>
+      <parent link="${parent}"/>
+      <child link="base_link"/>
     </joint>
     <link name="base_link">
       <visual>
         <geometry>
-          <mesh filename="package://walkie_description/meshes/walkie/base_link.dae" />
-            <!-- scale="0.001 0.001 0.001" /> -->
+          <!-- <mesh filename="package://walkie_description/meshes/walkie/base_link.dae"/> -->
+          <mesh filename="package://walkie_description/meshes/walkie/base_link.stl" scale="0.001 0.001 0.001"/>
         </geometry>
-        <material name="white" />
+        <material name="grey"/>
       </visual>
       <collision>
         <geometry>
-          <mesh filename="package://walkie_description/meshes/walkie/base_link_collision_fix_origin.stl" />
-            <!-- scale="0.001 0.001 0.001" /> -->
+          <mesh filename="package://walkie_description/meshes/walkie/base_link_collision.stl"/>
         </geometry>
       </collision>
-      <xacro:inertial_cylinder mass="${base_mass}" length="${bass_thickness}"
-        radius="${base_radian}">
-        <origin xyz="0 0 0" rpy="0 0 0" />
+      <xacro:inertial_cylinder mass="${base_mass}" length="${bass_thickness}" radius="${base_radian}">
+        <origin xyz="0 0 0" rpy="0 0 0"/>
       </xacro:inertial_cylinder>
-      <!-- <inertial>
-		<origin xyz="0 0 0"/>
-		<mass value="1.167"/>
-		<inertia ixx="0.0016" ixy="0" ixz="0" iyy="0.0016" iyz="0" izz="0.0032" />
-	  </inertial> -->
     </link>
   </xacro:macro>

File: urdf/walkie/omni_wheel/gz_omni_wheel.urdf.xacro (robot description, xacro)
@@ -1,112 +1,79 @@
 <?xml version="1.0"?>
 <robot xmlns:xacro="http://ros.org/wiki/xacro">
-    <xacro:include filename="$(find walkie_description)/urdf/inertial_macros.xacro" />
-    <xacro:include filename="$(find walkie_description)/urdf/walkie/omni_wheel/omni_wheel.gazebo.xacro" />
-    <xacro:include filename="$(find walkie_description)/urdf/walkie/omni_wheel/omni_wheel.transmission.xacro" />
-    <xacro:include filename="$(find walkie_description)/urdf/walkie/roller/gz_roller.urdf.xacro" />
-    <xacro:property name="wheel_thickness" value="0.0185" />
-    <xacro:property name="wheel_radian" value="0.0175" />
-    <xacro:property name="wheel_mass" value="0.05" />
-    <xacro:macro name="wheel_v0" params="prefix parent *joint_origin *joint_axis">
-        <joint name="${prefix}_wheel_joint" type="continuous">
-            <xacro:insert_block name="joint_origin" />
-            <parent link="${parent}" />
-            <child link="${prefix}_wheel_link" />
-            <limit effort="100" velocity="100" />
-            <dynamics damping="5.0" friction="0.5"/>
-            <xacro:insert_block name="joint_axis" />
-        </joint>
-        <link name="${prefix}_wheel_link">
-            <visual>
-                <geometry>
-                    <mesh filename="package://walkie_description/meshes/walkie/omni_wheel.dae"
-                        scale="1 1 1" />
-                </geometry>
-            </visual>
-            <xacro:inertial_cylinder mass="${wheel_mass}" length="${wheel_thickness}"
-                radius="${wheel_radian}">
-                <origin xyz="0 ${wheel_thickness/2} 0" rpy="1.570796327 0 0" />
-            </xacro:inertial_cylinder>
-        </link>
-        <xacro:roller prefix="${prefix}" num="1">
-            <origin xyz="0.057 0.0139 0.0" rpy="0.0 0.0 0.0" />
-            <axis xyz="0.0 0.0 1.0" />
-        </xacro:roller>
-        <xacro:roller prefix="${prefix}" num="2">
-            <origin xyz="0.0494 0.0139 0.0285" rpy="0.0 0.0 0.0" />
-            <axis xyz="-0.5 0.0 0.866025" />
-        </xacro:roller>
-        <xacro:roller prefix="${prefix}" num="3">
-            <origin xyz="0.0285 0.0139 0.0494" rpy="0.0 0.0 0.0" />
-            <axis xyz="-0.866025 0.0 0.5" />
-        </xacro:roller>
-        <xacro:roller prefix="${prefix}" num="4">
-            <origin xyz="0.0 0.0139 0.057" rpy="0.0 0.0 0.0" />
-            <axis xyz="-1.0 0.0 0.0" />
-        </xacro:roller>
-        <xacro:roller prefix="${prefix}" num="5">
-            <origin xyz="-0.0285 0.0139 0.0494" rpy="0.0 0.0 0.0" />
-            <axis xyz="-0.866025 0.0 -0.5" />
-        </xacro:roller>
-        <xacro:roller prefix="${prefix}" num="6">
-            <origin xyz="-0.0494 0.0139 0.0285" rpy="0.0 0.0 0.0" />
-            <axis xyz="-0.5 0.0 -0.866025" />
-        </xacro:roller>
-        <xacro:roller prefix="${prefix}" num="7">
-            <origin xyz="-0.057 0.0139 0.0" rpy="0.0 0.0 0.0" />
-            <axis xyz="-0.0 0.0 -1.0" />
-        </xacro:roller>
-        <xacro:roller prefix="${prefix}" num="8">
-            <origin xyz="-0.0494 0.0139 -0.0285" rpy="0.0 0.0 0.0" />
-            <axis xyz="0.5 0.0 -0.866025" />
-        </xacro:roller>
-        <xacro:roller prefix="${prefix}" num="9">
-            <origin xyz="-0.0285 0.0139 -0.0494" rpy="0.0 0.0 0.0" />
-            <axis xyz="0.866025 0.0 -0.5" />
-        </xacro:roller>
-        <xacro:roller prefix="${prefix}" num="10">
-            <origin xyz="-0.0 0.0139 -0.057" rpy="0.0 0.0 0.0" />
-            <axis xyz="1.0 0.0 -0.0" />
-        </xacro:roller>
-        <xacro:roller prefix="${prefix}" num="11">
-            <origin xyz="0.0285 0.0139 -0.0494" rpy="0.0 0.0 0.0" />
-            <axis xyz="0.866025 0.0 0.5" />
-        </xacro:roller>
-        <xacro:roller prefix="${prefix}" num="12">
-            <origin xyz="0.0494 0.0139 -0.0285" rpy="0.0 0.0 0.0" />
-            <axis xyz="0.5 0.0 0.866025" />
-        </xacro:roller>
-        <!-- <xacro:roller prefix="${prefix}" num="1"> -->
-            <!-- <origin xyz="0.0055 0.0046 0.0" rpy="0.0 0.0 0.0" /> -->
-            <!-- <axis xyz="0.0 0.0 1.0" /> -->
-        <!-- </xacro:roller> -->
-        <!-- <xacro:roller prefix="${prefix}" num="2"> -->
-            <!-- <origin xyz="0.0 0.0046 0.0055" rpy="0.0 0.0 0.0" /> -->
-            <!-- <axis xyz="-1.0 0.0 0.0" /> -->
-        <!-- </xacro:roller> -->
-        <!-- <xacro:roller prefix="${prefix}" num="3"> -->
-            <!-- <origin xyz="-0.0055 0.0046 0.0" rpy="0.0 0.0 0.0" /> -->
-            <!-- <axis xyz="-0.0 0.0 -1.0" /> -->
-        <!-- </xacro:roller> -->
-        <!-- <xacro:roller prefix="${prefix}" num="4"> -->
-            <!-- <origin xyz="-0.0 0.0046 -0.0055" rpy="0.0 0.0 0.0" /> -->
-            <!-- <axis xyz="1.0 0.0 -0.0" /> -->
-        <!-- </xacro:roller> -->
-        <!-- <xacro:roller prefix="${prefix}" num="5"> -->
-            <!-- <origin xyz="0.0039 0.0139 0.0039" rpy="0.0 0.0 0.0" /> -->
-            <!-- <axis xyz="-0.707107 0.0 0.707107" /> -->
-        <!-- </xacro:roller> -->
-        <!-- <xacro:roller prefix="${prefix}" num="6"> -->
-            <!-- <origin xyz="-0.0039 0.0139 0.0039" rpy="0.0 0.0 0.0" /> -->
-            <!-- <axis xyz="-0.707107 0.0 -0.707107" /> -->
-        <!-- </xacro:roller> -->
-        <!-- <xacro:roller prefix="${prefix}" num="7"> -->
-            <!-- <origin xyz="-0.0039 0.0139 -0.0039" rpy="0.0 0.0 0.0" /> -->
-            <!-- <axis xyz="0.707107 0.0 -0.707107" /> -->
-        <!-- </xacro:roller> -->
-        <!-- <xacro:roller prefix="${prefix}" num="8"> -->
-            <!-- <origin xyz="0.0039 0.0139 -0.0039" rpy="0.0 0.0 0.0" /> -->
-            <!-- <axis xyz="0.707107 0.0 0.707107" /> -->
-        <!-- </xacro:roller> -->
-    </xacro:macro>
+  <xacro:include filename="$(find walkie_description)/urdf/inertial_macros.xacro"/>
+  <xacro:include filename="$(find walkie_description)/urdf/walkie/omni_wheel/omni_wheel.gazebo.xacro"/>
+  <xacro:include filename="$(find walkie_description)/urdf/walkie/omni_wheel/omni_wheel.transmission.xacro"/>
+  <xacro:include filename="$(find walkie_description)/urdf/walkie/roller/gz_roller.urdf.xacro"/>
+  <xacro:property name="wheel_thickness" value="0.0185"/>
+  <xacro:property name="wheel_radian" value="0.0175"/>
+  <xacro:property name="wheel_mass" value="0.05"/>
+  <xacro:macro name="wheel_v0" params="prefix parent *joint_origin *joint_axis">
+    <joint name="${prefix}_wheel_joint" type="continuous">
+      <xacro:insert_block name="joint_origin"/>
+      <parent link="${parent}"/>
+      <child link="${prefix}_wheel_link"/>
+      <limit effort="100" velocity="100"/>
+      <dynamics damping="5.0" friction="0.5"/>
+      <xacro:insert_block name="joint_axis"/>
+    </joint>
+    <link name="${prefix}_wheel_link">
+      <visual>
+        <geometry>
+          <mesh filename="package://walkie_description/meshes/walkie/omni_wheel.dae" scale="1 1 1"/>
+          <!-- <mesh filename="package://walkie_description/meshes/walkie/omni_wheel.stl" scale="1 1 1"/> -->
+        </geometry>
+      </visual>
+      <xacro:inertial_cylinder mass="${wheel_mass}" length="${wheel_thickness}" radius="${wheel_radian}">
+        <origin xyz="0 ${wheel_thickness/2} 0" rpy="1.570796327 0 0"/>
+      </xacro:inertial_cylinder>
+    </link>
+    <xacro:roller prefix="${prefix}" num="1">
+      <origin xyz="0.0577 0.012 0.0" rpy="0.0 -0.0 0.0"/>
+      <axis xyz="0.0 0.0 1.0"/>
+    </xacro:roller>
+    <xacro:roller prefix="${prefix}" num="2">
+      <origin xyz="0.05 0.012 0.0289" rpy="0.0 -0.5236 0.0"/>
+      <axis xyz="0.0 0.0 1.0"/>
+    </xacro:roller>
+    <xacro:roller prefix="${prefix}" num="3">
+      <origin xyz="0.0289 0.012 0.05" rpy="0.0 -1.0472 0.0"/>
+      <axis xyz="0.0 0.0 1.0"/>
+    </xacro:roller>
+    <xacro:roller prefix="${prefix}" num="4">
+      <origin xyz="0.0 0.012 0.0577" rpy="0.0 -1.5708 0.0"/>
+      <axis xyz="0.0 0.0 1.0"/>
+    </xacro:roller>
+    <xacro:roller prefix="${prefix}" num="5">
+      <origin xyz="-0.0289 0.012 0.05" rpy="0.0 -2.0944 0.0"/>
+      <axis xyz="0.0 0.0 1.0"/>
+    </xacro:roller>
+    <xacro:roller prefix="${prefix}" num="6">
+      <origin xyz="-0.05 0.012 0.0289" rpy="0.0 -2.618 0.0"/>
+      <axis xyz="0.0 0.0 1.0"/>
+    </xacro:roller>
+    <xacro:roller prefix="${prefix}" num="7">
+      <origin xyz="-0.0577 0.012 0.0" rpy="0.0 -3.1416 0.0"/>
+      <axis xyz="0.0 0.0 1.0"/>
+    </xacro:roller>
+    <xacro:roller prefix="${prefix}" num="8">
+      <origin xyz="-0.05 0.012 -0.0289" rpy="0.0 -3.6652 0.0"/>
+      <axis xyz="0.0 0.0 1.0"/>
+    </xacro:roller>
+    <xacro:roller prefix="${prefix}" num="9">
+      <origin xyz="-0.0289 0.012 -0.05" rpy="0.0 -4.1888 0.0"/>
+      <axis xyz="0.0 0.0 1.0"/>
+    </xacro:roller>
+    <xacro:roller prefix="${prefix}" num="10">
+      <origin xyz="-0.0 0.012 -0.0577" rpy="0.0 -4.7124 0.0"/>
+      <axis xyz="0.0 0.0 1.0"/>
+    </xacro:roller>
+    <xacro:roller prefix="${prefix}" num="11">
+      <origin xyz="0.0289 0.012 -0.05" rpy="0.0 -5.236 0.0"/>
+      <axis xyz="0.0 0.0 1.0"/>
+    </xacro:roller>
+    <xacro:roller prefix="${prefix}" num="12">
+      <origin xyz="0.05 0.012 -0.0289" rpy="0.0 -5.7596 0.0"/>
+      <axis xyz="0.0 0.0 1.0"/>
+    </xacro:roller>
+  </xacro:macro>
 </robot>

File: urdf/walkie/roller/gz_roller.urdf.xacro (robot description, xacro)
@@ -1,37 +1,28 @@
 <?xml version="1.0"?>
 <robot xmlns:xacro="http://ros.org/wiki/xacro">
-    <xacro:include filename="$(find walkie_description)/urdf/inertial_macros.xacro" />
-    <xacro:include filename="$(find walkie_description)/urdf/walkie/roller/roller.gazebo.xacro" />
-    <xacro:property name="roller_mass" value="0.0001" />
-    <xacro:property name="roller_radius" value="0.019" />
-    <xacro:macro name="roller" params="prefix num *joint_origin *joint_axis">
-        <link name="roller_${prefix}_${num}_link">
-            <xacro:inertial_sphere mass="${roller_mass}" radius="${roller_radius}">
-                <origin xyz="0 0 0" rpy="0 0 0" />
-            </xacro:inertial_sphere>
-            <collision>
-                <origin xyz="0 0 0" rpy="0 0 0" />
-                <geometry>
-                    <sphere radius="${roller_radius}" />
-                  <!-- <mesh filename="package://armmy_omnibot/meshes/omni_wheel/Roller_Simplyfier.stl" -->
-                    <!-- scale="0.001 0.001 0.001" /> -->
-                  <!-- <mesh filename="$(find walkie_description)/meshes/walkie/roller_simplify.stl" -->
-                  <!-- <mesh filename="package://walkie_description/meshes/walkie/roller_simplify_z.stl" -->
-                      <!-- optimization="convex_decomposition"> -->
-                        <!-- <convex_decomposition> -->
-                            <!-- <voxel_resolution>500000</voxel_resolution> -->
-                            <!-- <max_convex_hulls>16</max_convex_hulls> -->
-                        <!-- </convex_decomposition> -->
-                      <!-- </mesh> -->
-                </geometry>
-            </collision>
-        </link>
-        <joint name="roller_${prefix}_${num}_joint" type="continuous">
-            <xacro:insert_block name="joint_origin" />
-            <parent link="${prefix}_wheel_link" />
-            <child link="roller_${prefix}_${num}_link" />
-            <xacro:insert_block name="joint_axis" />
-        </joint>
-        <xacro:roller_gazebo_v0 prefix="${prefix}" />
-    </xacro:macro>
+  <xacro:include filename="$(find walkie_description)/urdf/inertial_macros.xacro"/>
+  <xacro:include filename="$(find walkie_description)/urdf/walkie/roller/roller.gazebo.xacro"/>
+  <xacro:property name="roller_mass" value="0.0001"/>
+  <xacro:property name="roller_radius" value="0.019"/>
+  <xacro:macro name="roller" params="prefix num *joint_origin *joint_axis">
+    <link name="roller_${prefix}_${num}_link">
+      <xacro:inertial_sphere mass="${roller_mass}" radius="${roller_radius}">
+        <origin xyz="0 0 0" rpy="0 0 0"/>
+      </xacro:inertial_sphere>
+      <collision>
+        <origin xyz="0 0 0" rpy="0 0 0"/>
+        <geometry>
+          <!-- <sphere radius="${roller_radius}"/> -->
+          <cylinder length="0.005" radius="${roller_radius}"/>
+        </geometry>
+      </collision>
+    </link>
+    <joint name="roller_${prefix}_${num}_joint" type="continuous">
+      <xacro:insert_block name="joint_origin"/>
+      <parent link="${prefix}_wheel_link"/>
+      <child link="roller_${prefix}_${num}_link"/>
+      <xacro:insert_block name="joint_axis"/>
+    </joint>
+    <xacro:roller_gazebo_v0 prefix="${prefix}"/>
+  </xacro:macro>
 </robot>
