Commit message: change frictioness of model

File: robots/gz_walkie.urdf.xacro (robot description, xacro)
@@ -3,10 +3,9 @@
   <xacro:property name="M_PI" value="3.14159274" />
   <xacro:arg name="use_ros2_control" default="true" />
-  <xacro:arg name="sim_mode" default="false" />
+  <xacro:arg name="sim_mode" default="true" />
   <xacro:include filename="$(find walkie_description)/urdf/walkie/base/base.urdf.xacro" />
   <xacro:include filename="$(find walkie_description)/urdf/walkie/omni_wheel/gz_omni_wheel.urdf.xacro" />
   <!-- <xacro:include filename="$(find walkie_description)/urdf/lidar/lidar_gz.urdf.xacro" /> -->
   <!-- <xacro:include filename="$(find walkie_description)/urdf/imu/imu_gz.urdf.xacro" /> -->
-  <!-- <xacro:include filename="$(find walkie_description)/urdf/color.xacro" /> -->
   <!-- =============== Link & Joint =============== -->
   <!-- Base -->
@@ -15,22 +14,23 @@
     <origin xyz="0 0 0" rpy="0 0 ${M_PI / 4}" />
   </xacro:base_v0>
+  <xacro:base_gazebo_v0 />
   <!-- Wheel -->
   <!-- 1st wheel -->
-  <xacro:wheel_v0 prefix="b_l" parent="base_link">
+  <xacro:wheel_v0 prefix="bl" parent="base_link">
     <origin xyz="0.177622395 0.177622395 0.05" rpy="0 0 -${M_PI/4}" />
     <axis xyz="0.0 1.0 0.0" />
   </xacro:wheel_v0>
   <!-- 2nd wheel -->
-  <xacro:wheel_v0 prefix="b_r" parent="base_link">
+  <xacro:wheel_v0 prefix="br" parent="base_link">
     <origin xyz="-0.177622395 0.177622395 0.05" rpy="0 0 -${3*M_PI/4}" />
     <axis xyz="0.0 1.0 0.0" />
   </xacro:wheel_v0>
   <!-- 3rd wheel -->
-  <xacro:wheel_v0 prefix="f_r" parent="base_link">
+  <xacro:wheel_v0 prefix="fr" parent="base_link">
     <origin xyz="-0.177622395 -0.177622395 0.05" rpy="0 0 -${5*M_PI/4}" />
     <axis xyz="0.0 1.0 0.0" />
   </xacro:wheel_v0>
   <!-- 4th wheel -->
-  <xacro:wheel_v0 prefix="f_l" parent="base_link">
+  <xacro:wheel_v0 prefix="fl" parent="base_link">
     <origin xyz="0.177622395 -0.177622395 0.05" rpy="0 0 -${7*M_PI/4}" />
     <axis xyz="0.0 1.0 0.0" />
@@ -46,66 +46,6 @@
   <!-- </xacro:imu_v0> -->
   <!-- <xacro:imu_gazebo_v0 prefix="top" /> -->
-  <!-- ===============  Transmission =============== -->
-  <!-- <xacro:wheel_trans_v0 prefix="b_l" /> -->
-  <xacro:wheel_trans_v0 prefix="b_r" />
-  <!-- </xacro:imu_v0-> -->
-  <!-- <xacro:imu_gazebo_v0 prefix="top" /> -->
-  <!-- Base -->
-  <!-- <xacro:base_gazebo_v0 /> -->
-  <!-- Wheel -->
-  <!-- <xacro:wheel_gazebo_v0 prefix="b_l" /> -->
-  <xacro:wheel_gazebo_v0 prefix="b_r" />
-  <!-- Base -->
-  <!--- <xacro:base_gazebo_v0 /> -->
-  <!-- <ros2_control name="GazeboSystem" type="system"> -->
-    <!-- <hardware> -->
-      <!-- <plugin>gz_ros2_control/GazeboSimSystem</plugin> -->
-    <!-- </hardware> -->
-    <!-- <joint name="b_l_wheel_joint"> -->
-      <!-- <command_interface name="velocity"> -->
-        <!-- <param name="min">-3.14</param> -->
-        <!-- <param name="max">3.14</param> -->
-      <!-- </command_interface> -->
-      <!-- <state_interface name="velocity" /> -->
-      <!-- <state_interface name="position" /> -->
-    <!-- </joint> -->
-    <!-- <joint name="b_r_wheel_joint"> -->
-      <!-- </command_interface> -->
-    -  <!-- <state_interface name="velocity" /> -->
-        <!-- <param name="max">3.14</param> -->
-      <!-- </command_interface> -->
-      <!-- <state_interface name="velocity" /> -->
-      <!-- <state_interface name="position" /> -->
-    <!-- </joint> -->
-    <!-- <joint name="third_wheel_joint"> -->
-      <!-- <command_interface name="velocity"> -->
-        <!-- <param name="min">-3.14</param> -->
-        <!-- <param name="max">3.14</param> -->
-      <!-- </command_interface> -->
-      <!-- <state_interface name="velocity" /> -->
-      <!-- <state_interface name="position" /> -->
-    <!-- </joint> -->
-    <!-- <joint name="fourth_wheel_joint"> -->
-      <!-- <command_interface name="velocity"> -->
-        <!-- <param name="min">-3.14</param> -->
-        <!-- <param name="max">3.14</param> -->
-      <!-- </command_interface> -->
-      <!-- <state_interface name="velocity" /> -->
-      <!-- <state_interface name="position" /> -->
-    <!-- </joint> -->
-  <!-- </ros2_control> -->
-  <!-- <gazebo> -->
-    <!-- <plugin name="gz_ros2_control::GazeboSimROS2ControlPlugin" -->
-      <!-- filename="libgz_ros2_control-system.so"> -->
-      <!-- <parameters>$(find walkie_description)/config/ros2_controller/my_controllers.yaml</parameters> -->
-    <!-- </plugin> -->
-    <!-- <plugin filename="libignition-gazebo6-pose-publisher-system.so" -->
-      <!-- name="ignition::gazebo::systems::PosePublisher"> -->
-      <!-- <publish_model_pose>true</publish_model_pose> -->
-      <!-- <publish_link_pose>false</publish_link_pose> -->
-      <!-- <publish_nested_model_pose>true</publish_nested_model_pose> -->
-      <!-- <static_publisher>true</static_publisher> -->
-      <!-- <static_update_frequency>10</static_update_frequency> -->
-   <!-- </plugin> -->
-  <!-- </gazebo> -->
+  <xacro:if value="$(arg use_ros2_control)">
+    <xacro:include filename="$(find walkie_description)/urdf/walkie/ros2_control.xacro"/>
+  </xacro:if>
 </robot>

File: urdf/walkie/omni_wheel/gz_omni_wheel.urdf.xacro (robot description, xacro)
@@ -30,34 +30,130 @@
         </link>
         <xacro:roller prefix="${prefix}" num="1">
-            <origin xyz="0.0055 0.00925 0.0" rpy="0.0 0.0 0.0" />
+            <origin xyz="0.057 0.0139 0.0" rpy="0.0 0.0 0.0" />
             <axis xyz="0.0 0.0 1.0" />
         </xacro:roller>
         <xacro:roller prefix="${prefix}" num="2">
-            <origin xyz="0.0 0.00925 0.0055" rpy="0.0 0.0 0.0" />
-            <axis xyz="-1.0 0.0 0.0" />
+            <origin xyz="0.0559 0.0139 0.0111" rpy="0.0 0.0 0.0" />
+            <axis xyz="-0.19509 0.0 0.980785" />
         </xacro:roller>
         <xacro:roller prefix="${prefix}" num="3">
-            <origin xyz="-0.0055 0.00925 0.0" rpy="0.0 0.0 0.0" />
-            <axis xyz="-0.0 0.0 -1.0" />
+            <origin xyz="0.0527 0.0139 0.0218" rpy="0.0 0.0 0.0" />
+            <axis xyz="-0.382683 0.0 0.92388" />
         </xacro:roller>
         <xacro:roller prefix="${prefix}" num="4">
-            <origin xyz="-0.0 0.00925 -0.0055" rpy="0.0 0.0 0.0" />
-            <axis xyz="1.0 0.0 -0.0" />
+            <origin xyz="0.0474 0.0139 0.0317" rpy="0.0 0.0 0.0" />
+            <axis xyz="-0.55557 0.0 0.83147" />
         </xacro:roller>
         <xacro:roller prefix="${prefix}" num="5">
-            <origin xyz="0.0039 0.00925 0.0039" rpy="0.0 0.0 0.0" />
+            <origin xyz="0.0403 0.0139 0.0403" rpy="0.0 0.0 0.0" />
             <axis xyz="-0.707107 0.0 0.707107" />
         </xacro:roller>
         <xacro:roller prefix="${prefix}" num="6">
-            <origin xyz="-0.0039 0.00925 0.0039" rpy="0.0 0.0 0.0" />
+            <origin xyz="0.0317 0.0139 0.0474" rpy="0.0 0.0 0.0" />
+            <axis xyz="-0.83147 0.0 0.55557" />
+        </xacro:roller>
+        <xacro:roller prefix="${prefix}" num="7">
+            <origin xyz="0.0218 0.0139 0.0527" rpy="0.0 0.0 0.0" />
+            <axis xyz="-0.92388 0.0 0.382683" />
+        </xacro:roller>
+        <xacro:roller prefix="${prefix}" num="8">
+            <origin xyz="0.0111 0.0139 0.0559" rpy="0.0 0.0 0.0" />
+            <axis xyz="-0.980785 0.0 0.19509" />
+        </xacro:roller>
+        <xacro:roller prefix="${prefix}" num="9">
+            <origin xyz="0.0 0.0139 0.057" rpy="0.0 0.0 0.0" />
+            <axis xyz="-1.0 0.0 0.0" />
+        </xacro:roller>
+        <xacro:roller prefix="${prefix}" num="10">
+            <origin xyz="-0.0111 0.0139 0.0559" rpy="0.0 0.0 0.0" />
+            <axis xyz="-0.980785 0.0 -0.19509" />
+        </xacro:roller>
+        <xacro:roller prefix="${prefix}" num="11">
+            <origin xyz="-0.0218 0.0139 0.0527" rpy="0.0 0.0 0.0" />
+            <axis xyz="-0.92388 0.0 -0.382683" />
+        </xacro:roller>
+        <xacro:roller prefix="${prefix}" num="12">
+            <origin xyz="-0.0317 0.0139 0.0474" rpy="0.0 0.0 0.0" />
+            <axis xyz="-0.83147 0.0 -0.55557" />
+        </xacro:roller>
+        <xacro:roller prefix="${prefix}" num="13">
+            <origin xyz="-0.0403 0.0139 0.0403" rpy="0.0 0.0 0.0" />
             <axis xyz="-0.707107 0.0 -0.707107" />
         </xacro:roller>
-        <xacro:roller prefix="${prefix}" num="7">
-            <origin xyz="-0.0039 0.00925 -0.0039" rpy="0.0 0.0 0.0" />
+        <xacro:roller prefix="${prefix}" num="14">
+            <origin xyz="-0.0474 0.0139 0.0317" rpy="0.0 0.0 0.0" />
+            <axis xyz="-0.55557 0.0 -0.83147" />
+        </xacro:roller>
+        <xacro:roller prefix="${prefix}" num="15">
+            <origin xyz="-0.0527 0.0139 0.0218" rpy="0.0 0.0 0.0" />
+            <axis xyz="-0.382683 0.0 -0.92388" />
+        </xacro:roller>
+        <xacro:roller prefix="${prefix}" num="16">
+            <origin xyz="-0.0559 0.0139 0.0111" rpy="0.0 0.0 0.0" />
+            <axis xyz="-0.19509 0.0 -0.980785" />
+        </xacro:roller>
+        <xacro:roller prefix="${prefix}" num="17">
+            <origin xyz="-0.057 0.0139 0.0" rpy="0.0 0.0 0.0" />
+            <axis xyz="-0.0 0.0 -1.0" />
+        </xacro:roller>
+        <xacro:roller prefix="${prefix}" num="18">
+            <origin xyz="-0.0559 0.0139 -0.0111" rpy="0.0 0.0 0.0" />
+            <axis xyz="0.19509 0.0 -0.980785" />
+        </xacro:roller>
+        <xacro:roller prefix="${prefix}" num="19">
+            <origin xyz="-0.0527 0.0139 -0.0218" rpy="0.0 0.0 0.0" />
+            <axis xyz="0.382683 0.0 -0.92388" />
+        </xacro:roller>
+        <xacro:roller prefix="${prefix}" num="20">
+            <origin xyz="-0.0474 0.0139 -0.0317" rpy="0.0 0.0 0.0" />
+            <axis xyz="0.55557 0.0 -0.83147" />
+        </xacro:roller>
+        <xacro:roller prefix="${prefix}" num="21">
+            <origin xyz="-0.0403 0.0139 -0.0403" rpy="0.0 0.0 0.0" />
             <axis xyz="0.707107 0.0 -0.707107" />
         </xacro:roller>
-        <xacro:roller prefix="${prefix}" num="8">
-            <origin xyz="0.0039 0.00925 -0.0039" rpy="0.0 0.0 0.0" />
+        <xacro:roller prefix="${prefix}" num="22">
+            <origin xyz="-0.0317 0.0139 -0.0474" rpy="0.0 0.0 0.0" />
+            <axis xyz="0.83147 0.0 -0.55557" />
+        </xacro:roller>
+        <xacro:roller prefix="${prefix}" num="23">
+            <origin xyz="-0.0218 0.0139 -0.0527" rpy="0.0 0.0 0.0" />
+            <axis xyz="0.92388 0.0 -0.382683" />
+        </xacro:roller>
+        <xacro:roller prefix="${prefix}" num="24">
+            <origin xyz="-0.0111 0.0139 -0.0559" rpy="0.0 0.0 0.0" />
+            <axis xyz="0.980785 0.0 -0.19509" />
+        </xacro:roller>
+        <xacro:roller prefix="${prefix}" num="25">
+            <origin xyz="-0.0 0.0139 -0.057" rpy="0.0 0.0 0.0" />
+            <axis xyz="1.0 0.0 -0.0" />
+        </xacro:roller>
+        <xacro:roller prefix="${prefix}" num="26">
+            <origin xyz="0.0111 0.0139 -0.0559" rpy="0.0 0.0 0.0" />
+            <axis xyz="0.980785 0.0 0.19509" />
+        </xacro:roller>
+        <xacro:roller prefix="${prefix}" num="27">
+            <origin xyz="0.0218 0.0139 -0.0527" rpy="0.0 0.0 0.0" />
+            <axis xyz="0.92388 0.0 0.382683" />
+        </xacro:roller>
+        <xacro:roller prefix="${prefix}" num="28">
+            <origin xyz="0.0317 0.0139 -0.0474" rpy="0.0 0.0 0.0" />
+            <axis xyz="0.83147 0.0 0.55557" />
+        </xacro:roller>
+        <xacro:roller prefix="${prefix}" num="29">
+            <origin xyz="0.0403 0.0139 -0.0403" rpy="0.0 0.0 0.0" />
             <axis xyz="0.707107 0.0 0.707107" />
+        </xacro:roller>
+        <xacro:roller prefix="${prefix}" num="30">
+            <origin xyz="0.0474 0.0139 -0.0317" rpy="0.0 0.0 0.0" />
+            <axis xyz="0.55557 0.0 0.83147" />
+        </xacro:roller>
+        <xacro:roller prefix="${prefix}" num="31">
+            <origin xyz="0.0527 0.0139 -0.0218" rpy="0.0 0.0 0.0" />
+            <axis xyz="0.382683 0.0 0.92388" />
+        </xacro:roller>
+        <xacro:roller prefix="${prefix}" num="32">
+            <origin xyz="0.0559 0.0139 -0.0111" rpy="0.0 0.0 0.0" />
+            <axis xyz="0.19509 0.0 0.980785" />
         </xacro:roller>
         <!-- <xacro:roller prefix="${prefix}" num="1"> -->

File: urdf/walkie/omni_wheel/omni_wheel.transmission.xacro (robot description, xacro)
@@ -5,10 +5,10 @@
       <type>transmission_interface/SimpleTransmission</type>
       <joint name="${prefix}_wheel_joint">
-	<hardwareInterface>hardware_interface/VelocityJointInterface</hardwareInterface>
+        	<hardwareInterface>hardware_interface/VelocityJointInterface</hardwareInterface>
       </joint>
-	<actuator name="${prefix}_wheel_motor">
-	  <hardwareInterface>hardware_interface/VelocityJointInterface</hardwareInterface>
-	  <mechanicalReduction>30</mechanicalReduction>
-        </actuator>
+    	<actuator name="${prefix}_wheel_motor">
+    	  <hardwareInterface>hardware_interface/VelocityJointInterface</hardwareInterface>
+    	  <mechanicalReduction>30</mechanicalReduction>
+      </actuator>
     </transmission>
   </xacro:macro>

File: urdf/walkie/omni_wheel/omni_wheel.urdf.xacro (robot description, xacro)
@@ -22,12 +22,5 @@
             scale="1 1 1" />
         </geometry>
-        <!-- <material name="light_black" /> -->
       </visual>
-      <!-- <collision>
-        <geometry>
-          <mesh filename="package://armmy_omnibot/meshes/omni_wheel/wheel_base.stl"
-            scale="0.001 0.001 0.001" />
-        </geometry>
-      </collision> -->
       <xacro:inertial_cylinder mass="${wheel_mass}" length="${wheel_thickness}"
         radius="${wheel_radian}">
@@ -54,4 +47,8 @@
       </surface>
     </link>
+  <!-- --- Set Transmission --- -->
+  <xacro:wheel_trans_v0 prefix="${prefix}" />
+  <!-- --- Set Gazebo Params --- -->
+  <xacro:wheel_gazebo_v0 prefix="${prefix}"/>
   </xacro:macro>
 </robot>

File: urdf/walkie/roller/gz_roller.urdf.xacro (robot description, xacro)
@@ -2,6 +2,7 @@
 <robot xmlns:xacro="http://ros.org/wiki/xacro">
     <xacro:include filename="$(find walkie_description)/urdf/inertial_macros.xacro" />
+    <xacro:include filename="$(find walkie_description)/urdf/walkie/roller/roller.gazebo.xacro" />
     <xacro:property name="roller_mass" value="0.0001" />
-    <xacro:property name="roller_radius" value="0.012" />
+    <xacro:property name="roller_radius" value="0.019" />
     <xacro:macro name="roller" params="prefix num *joint_origin *joint_axis">
         <link name="roller_${prefix}_${num}_link">
@@ -15,5 +16,6 @@
                   <!-- <mesh filename="package://armmy_omnibot/meshes/omni_wheel/Roller_Simplyfier.stl" -->
                     <!-- scale="0.001 0.001 0.001" /> -->
-                  <!-- <mesh filename="package://armmy_omnibot/meshes/omni_wheel/Roller_Simplyfier.stl" -->
+                  <!-- <mesh filename="$(find walkie_description)/meshes/walkie/roller_simplify.stl" -->
+                  <!-- <mesh filename="package://walkie_description/meshes/walkie/roller_simplify_z.stl" -->
                       <!-- optimization="convex_decomposition"> -->
                         <!-- <convex_decomposition> -->
@@ -27,6 +29,6 @@
               <friction>
                 <ode>
-                  <mu1>1.2</mu1>
-                  <mu2>1.2</mu2>
+                  <mu1>2.2</mu1>
+                  <mu2>2.2</mu2>
                   <kp>1e15</kp>
                   <kd>1e13</kd>
@@ -39,5 +41,8 @@
               <contact>
                 <ode>
-                  <max_vel>10</max_vel>
+                    <min_depth>0.003</min_depth>
+                    <kp>1e6</kp>
+                    <kd>1.0</kd>
+                    <max_vel>10</max_vel>
                 </ode>
               </contact>
@@ -65,4 +70,5 @@
             <xacro:insert_block name="joint_axis" />
         </joint>
+        <xacro:roller_gazebo_v0 prefix="${prefix}" />
     </xacro:macro>
 </robot>

File: urdf/walkie/roller/roller.gazebo.xacro (robot description, xacro)
@@ -3,5 +3,5 @@
   <xacro:macro name="roller_gazebo_v0" params="prefix">
     <gazebo reference="${prefix}_roller_link">
-      <!-- <selfCollide>false</selfCollide> -->
+      <selfCollide>false</selfCollide>
       <mu value="8.8" />
       <mu2 value="1.2" />

File: urdf/walkie/roller/roller.urdf.xacro (robot description, xacro)
@@ -25,6 +25,5 @@
       <collision>
         <geometry>
-          <mesh filename="package://armmy_omnibot/meshes/omni_wheel/Roller_Simplyfier.stl"
-            scale="0.001 0.001 0.001" />
+          <mesh filename="package://armmy_omnibot/meshes/omni_wheel/Roller_Simplyfier.stl" />
         </geometry>
       </collision>
