Commit message: finish add forward velocity control for wheel joints

File: robots/gz_walkie.urdf.xacro (robot description, xacro)
@@ -12,5 +12,5 @@
   <link name="base_footprint" />
   <xacro:base_v0 parent="base_footprint">
-    <origin xyz="0 0 0" rpy="0 0 ${M_PI / 4}" />
+    <origin xyz="0 0 0" rpy="0 0 ${M_PI / 2}" />
   </xacro:base_v0>
   <xacro:base_gazebo_v0 />
@@ -23,15 +23,15 @@
   <!-- 2nd wheel -->
   <xacro:wheel_v0 prefix="br" parent="base_link">
-    <origin xyz="-0.177622395 0.177622395 0.05" rpy="0 0 -${3*M_PI/4}" />
+    <origin xyz="-0.177622395 0.177622395 0.05" rpy="0 0 ${M_PI/4}" />
     <axis xyz="0.0 1.0 0.0" />
   </xacro:wheel_v0>
   <!-- 3rd wheel -->
   <xacro:wheel_v0 prefix="fr" parent="base_link">
-    <origin xyz="-0.177622395 -0.177622395 0.05" rpy="0 0 -${5*M_PI/4}" />
+    <origin xyz="-0.177622395 -0.177622395 0.05" rpy="0 0 ${3*M_PI/4}" />
     <axis xyz="0.0 1.0 0.0" />
   </xacro:wheel_v0>
   <!-- 4th wheel -->
   <xacro:wheel_v0 prefix="fl" parent="base_link">
-    <origin xyz="0.177622395 -0.177622395 0.05" rpy="0 0 -${7*M_PI/4}" />
+    <origin xyz="0.177622395 -0.177622395 0.05" rpy="0 0 ${5*M_PI/4}" />
     <axis xyz="0.0 1.0 0.0" />
   </xacro:wheel_v0>

File: urdf/walkie/base/base.urdf.xacro (robot description, xacro)
@@ -22,5 +22,5 @@
       <collision>
         <geometry>
-          <mesh filename="package://walkie_description/meshes/walkie/base_link_collision.stl" />
+          <mesh filename="package://walkie_description/meshes/walkie/base_link_collision_fix_origin.stl" />
             <!-- scale="0.001 0.001 0.001" /> -->
         </geometry>

File: urdf/walkie/omni_wheel/gz_omni_wheel.urdf.xacro (robot description, xacro)
@@ -14,5 +14,5 @@
             <child link="${prefix}_wheel_link" />
             <limit effort="100" velocity="100" />
-            <dynamics damping="1.0" friction="0.5"/>
+            <dynamics damping="5.0" friction="0.5"/>
             <xacro:insert_block name="joint_axis" />
         </joint>
@@ -34,126 +34,46 @@
         </xacro:roller>
         <xacro:roller prefix="${prefix}" num="2">
-            <origin xyz="0.0559 0.0139 0.0111" rpy="0.0 0.0 0.0" />
-            <axis xyz="-0.19509 0.0 0.980785" />
+            <origin xyz="0.0494 0.0139 0.0285" rpy="0.0 0.0 0.0" />
+            <axis xyz="-0.5 0.0 0.866025" />
         </xacro:roller>
         <xacro:roller prefix="${prefix}" num="3">
-            <origin xyz="0.0527 0.0139 0.0218" rpy="0.0 0.0 0.0" />
-            <axis xyz="-0.382683 0.0 0.92388" />
+            <origin xyz="0.0285 0.0139 0.0494" rpy="0.0 0.0 0.0" />
+            <axis xyz="-0.866025 0.0 0.5" />
         </xacro:roller>
         <xacro:roller prefix="${prefix}" num="4">
-            <origin xyz="0.0474 0.0139 0.0317" rpy="0.0 0.0 0.0" />
-            <axis xyz="-0.55557 0.0 0.83147" />
-        </xacro:roller>
-        <xacro:roller prefix="${prefix}" num="5">
-            <origin xyz="0.0403 0.0139 0.0403" rpy="0.0 0.0 0.0" />
-            <axis xyz="-0.707107 0.0 0.707107" />
-        </xacro:roller>
-        <xacro:roller prefix="${prefix}" num="6">
-            <origin xyz="0.0317 0.0139 0.0474" rpy="0.0 0.0 0.0" />
-            <axis xyz="-0.83147 0.0 0.55557" />
-        </xacro:roller>
-        <xacro:roller prefix="${prefix}" num="7">
-            <origin xyz="0.0218 0.0139 0.0527" rpy="0.0 0.0 0.0" />
-            <axis xyz="-0.92388 0.0 0.382683" />
-        </xacro:roller>
-        <xacro:roller prefix="${prefix}" num="8">
-            <origin xyz="0.0111 0.0139 0.0559" rpy="0.0 0.0 0.0" />
-            <axis xyz="-0.980785 0.0 0.19509" />
-        </xacro:roller>
-        <xacro:roller prefix="${prefix}" num="9">
             <origin xyz="0.0 0.0139 0.057" rpy="0.0 0.0 0.0" />
             <axis xyz="-1.0 0.0 0.0" />
         </xacro:roller>
-        <xacro:roller prefix="${prefix}" num="10">
-            <origin xyz="-0.0111 0.0139 0.0559" rpy="0.0 0.0 0.0" />
-            <axis xyz="-0.980785 0.0 -0.19509" />
+        <xacro:roller prefix="${prefix}" num="5">
+            <origin xyz="-0.0285 0.0139 0.0494" rpy="0.0 0.0 0.0" />
+            <axis xyz="-0.866025 0.0 -0.5" />
         </xacro:roller>
-        <xacro:roller prefix="${prefix}" num="11">
-            <origin xyz="-0.0218 0.0139 0.0527" rpy="0.0 0.0 0.0" />
-            <axis xyz="-0.92388 0.0 -0.382683" />
+        <xacro:roller prefix="${prefix}" num="6">
+            <origin xyz="-0.0494 0.0139 0.0285" rpy="0.0 0.0 0.0" />
+            <axis xyz="-0.5 0.0 -0.866025" />
         </xacro:roller>
-        <xacro:roller prefix="${prefix}" num="12">
-            <origin xyz="-0.0317 0.0139 0.0474" rpy="0.0 0.0 0.0" />
-            <axis xyz="-0.83147 0.0 -0.55557" />
-        </xacro:roller>
-        <xacro:roller prefix="${prefix}" num="13">
-            <origin xyz="-0.0403 0.0139 0.0403" rpy="0.0 0.0 0.0" />
-            <axis xyz="-0.707107 0.0 -0.707107" />
-        </xacro:roller>
-        <xacro:roller prefix="${prefix}" num="14">
-            <origin xyz="-0.0474 0.0139 0.0317" rpy="0.0 0.0 0.0" />
-            <axis xyz="-0.55557 0.0 -0.83147" />
-        </xacro:roller>
-        <xacro:roller prefix="${prefix}" num="15">
-            <origin xyz="-0.0527 0.0139 0.0218" rpy="0.0 0.0 0.0" />
-            <axis xyz="-0.382683 0.0 -0.92388" />
-        </xacro:roller>
-        <xacro:roller prefix="${prefix}" num="16">
-            <origin xyz="-0.0559 0.0139 0.0111" rpy="0.0 0.0 0.0" />
-            <axis xyz="-0.19509 0.0 -0.980785" />
-        </xacro:roller>
-        <xacro:roller prefix="${prefix}" num="17">
+        <xacro:roller prefix="${prefix}" num="7">
             <origin xyz="-0.057 0.0139 0.0" rpy="0.0 0.0 0.0" />
             <axis xyz="-0.0 0.0 -1.0" />
         </xacro:roller>
-        <xacro:roller prefix="${prefix}" num="18">
-            <origin xyz="-0.0559 0.0139 -0.0111" rpy="0.0 0.0 0.0" />
-            <axis xyz="0.19509 0.0 -0.980785" />
+        <xacro:roller prefix="${prefix}" num="8">
+            <origin xyz="-0.0494 0.0139 -0.0285" rpy="0.0 0.0 0.0" />
+            <axis xyz="0.5 0.0 -0.866025" />
         </xacro:roller>
-        <xacro:roller prefix="${prefix}" num="19">
-            <origin xyz="-0.0527 0.0139 -0.0218" rpy="0.0 0.0 0.0" />
-            <axis xyz="0.382683 0.0 -0.92388" />
+        <xacro:roller prefix="${prefix}" num="9">
+            <origin xyz="-0.0285 0.0139 -0.0494" rpy="0.0 0.0 0.0" />
+            <axis xyz="0.866025 0.0 -0.5" />
         </xacro:roller>
-        <xacro:roller prefix="${prefix}" num="20">
-            <origin xyz="-0.0474 0.0139 -0.0317" rpy="0.0 0.0 0.0" />
-            <axis xyz="0.55557 0.0 -0.83147" />
-        </xacro:roller>
-        <xacro:roller prefix="${prefix}" num="21">
-            <origin xyz="-0.0403 0.0139 -0.0403" rpy="0.0 0.0 0.0" />
-            <axis xyz="0.707107 0.0 -0.707107" />
-        </xacro:roller>
-        <xacro:roller prefix="${prefix}" num="22">
-            <origin xyz="-0.0317 0.0139 -0.0474" rpy="0.0 0.0 0.0" />
-            <axis xyz="0.83147 0.0 -0.55557" />
-        </xacro:roller>
-        <xacro:roller prefix="${prefix}" num="23">
-            <origin xyz="-0.0218 0.0139 -0.0527" rpy="0.0 0.0 0.0" />
-            <axis xyz="0.92388 0.0 -0.382683" />
-        </xacro:roller>
-        <xacro:roller prefix="${prefix}" num="24">
-            <origin xyz="-0.0111 0.0139 -0.0559" rpy="0.0 0.0 0.0" />
-            <axis xyz="0.980785 0.0 -0.19509" />
-        </xacro:roller>
-        <xacro:roller prefix="${prefix}" num="25">
+        <xacro:roller prefix="${prefix}" num="10">
             <origin xyz="-0.0 0.0139 -0.057" rpy="0.0 0.0 0.0" />
             <axis xyz="1.0 0.0 -0.0" />
         </xacro:roller>
-        <xacro:roller prefix="${prefix}" num="26">
-            <origin xyz="0.0111 0.0139 -0.0559" rpy="0.0 0.0 0.0" />
-            <axis xyz="0.980785 0.0 0.19509" />
+        <xacro:roller prefix="${prefix}" num="11">
+            <origin xyz="0.0285 0.0139 -0.0494" rpy="0.0 0.0 0.0" />
+            <axis xyz="0.866025 0.0 0.5" />
         </xacro:roller>
-        <xacro:roller prefix="${prefix}" num="27">
-            <origin xyz="0.0218 0.0139 -0.0527" rpy="0.0 0.0 0.0" />
-            <axis xyz="0.92388 0.0 0.382683" />
-        </xacro:roller>
-        <xacro:roller prefix="${prefix}" num="28">
-            <origin xyz="0.0317 0.0139 -0.0474" rpy="0.0 0.0 0.0" />
-            <axis xyz="0.83147 0.0 0.55557" />
-        </xacro:roller>
-        <xacro:roller prefix="${prefix}" num="29">
-            <origin xyz="0.0403 0.0139 -0.0403" rpy="0.0 0.0 0.0" />
-            <axis xyz="0.707107 0.0 0.707107" />
-        </xacro:roller>
-        <xacro:roller prefix="${prefix}" num="30">
-            <origin xyz="0.0474 0.0139 -0.0317" rpy="0.0 0.0 0.0" />
-            <axis xyz="0.55557 0.0 0.83147" />
-        </xacro:roller>
-        <xacro:roller prefix="${prefix}" num="31">
-            <origin xyz="0.0527 0.0139 -0.0218" rpy="0.0 0.0 0.0" />
-            <axis xyz="0.382683 0.0 0.92388" />
-        </xacro:roller>
-        <xacro:roller prefix="${prefix}" num="32">
-            <origin xyz="0.0559 0.0139 -0.0111" rpy="0.0 0.0 0.0" />
-            <axis xyz="0.19509 0.0 0.980785" />
+        <xacro:roller prefix="${prefix}" num="12">
+            <origin xyz="0.0494 0.0139 -0.0285" rpy="0.0 0.0 0.0" />
+            <axis xyz="0.5 0.0 0.866025" />
         </xacro:roller>
         <!-- <xacro:roller prefix="${prefix}" num="1"> -->

File: urdf/walkie/roller/gz_roller.urdf.xacro (robot description, xacro)
@@ -26,41 +26,4 @@
                 </geometry>
             </collision>
-            <surface>
-              <friction>
-                <ode>
-                  <mu1>2.2</mu1>
-                  <mu2>2.2</mu2>
-                  <kp>1e15</kp>
-                  <kd>1e13</kd>
-                </ode>
-              </friction>
-              <bounce>
-                <restitution_coefficient>0.01</restitution_coefficient>
-                <threshold>0</threshold>
-              </bounce>
-              <contact>
-                <ode>
-                    <min_depth>0.003</min_depth>
-                    <kp>1e6</kp>
-                    <kd>1.0</kd>
-                    <max_vel>10</max_vel>
-                </ode>
-              </contact>
-            </surface>
-            <!-- <surface> -->
-                <!-- <friction> -->
-                    <!-- <ode> -->
-                        <!-- <mu>1.0</mu> -->
-                        <!-- <mu2>1.0</mu2> -->
-                    <!-- </ode> -->
-                <!-- </friction> -->
-                <!-- <contact> -->
-                    <!-- <ode> -->
-                        <!-- <min_depth>0.003</min_depth> -->
-                        <!-- <kp>1e6</kp> -->
-                        <!-- <kd>100</kd> -->
-                    <!-- </ode> -->
-                <!-- </contact> -->
-            <!-- </surface> -->
         </link>
         <joint name="roller_${prefix}_${num}_joint" type="continuous">

File: urdf/walkie/roller/roller.gazebo.xacro (robot description, xacro)
@@ -3,7 +3,27 @@
   <xacro:macro name="roller_gazebo_v0" params="prefix">
     <gazebo reference="${prefix}_roller_link">
-      <selfCollide>false</selfCollide>
-      <mu value="8.8" />
-      <mu2 value="1.2" />
+      <collision>
+        <surface>
+          <friction>
+            <ode>
+              <mu1>1.0</mu1>
+              <mu2>1.0</mu2>
+              <kp>1e15</kp>
+              <kd>1e13</kd>
+            </ode>
+          </friction>
+          <bounce>
+            <restitution_coefficient>0.01</restitution_coefficient>
+            <threshold>0</threshold>
+          </bounce>
+          <contact>
+            <ode>
+                <min_depth>0.005</min_depth>
+                <kp>1e6</kp>
+                <kd>1000</kd>
+            </ode>
+          </contact>
+        </surface>
+      </collision>
     </gazebo>
   </xacro:macro>

File: urdf/walkie/ros2_control.xacro (robot description, xacro)
@@ -2,5 +2,5 @@
 <robot xmlns:xacro="http://www.ros.org/wiki/xacro">
     <xacro:if value="$(arg sim_mode)">
-        <ros2_control name="GazeboSystem" type="system">
+        <ros2_control name="GazeboSimSystem" type="system">
           <hardware>
             <plugin>gz_ros2_control/GazeboSimSystem</plugin>

Commit message: add sensor

File: robots/gz_walkie.urdf.xacro (robot description, xacro)
@@ -4,8 +4,8 @@
   <xacro:arg name="use_ros2_control" default="true" />
   <xacro:arg name="sim_mode" default="true" />
-  <xacro:include filename="$(find walkie_description)/urdf/walkie/base/base.urdf.xacro" />
-  <xacro:include filename="$(find walkie_description)/urdf/walkie/omni_wheel/gz_omni_wheel.urdf.xacro" />
-  <!-- <xacro:include filename="$(find walkie_description)/urdf/lidar/lidar_gz.urdf.xacro" /> -->
-  <!-- <xacro:include filename="$(find walkie_description)/urdf/imu/imu_gz.urdf.xacro" /> -->
+  <xacro:include filename="$(find walkie_description)/urdf/walkie/base/base.urdf.xacro"/>
+  <xacro:include filename="$(find walkie_description)/urdf/walkie/omni_wheel/gz_omni_wheel.urdf.xacro"/>
+  <xacro:include filename="$(find walkie_description)/urdf/walkie/lidar/lidar_gz.urdf.xacro"/>
+  <xacro:include filename="$(find walkie_description)/urdf/walkie/imu/imu_gz.urdf.xacro"/>
   <!-- =============== Link & Joint =============== -->
   <!-- Base -->
@@ -37,13 +37,13 @@
   </xacro:wheel_v0>
   <!-- lidar sensor -->
-  <!-- <xacro:lidar_v0 prefix="top" parent="base_link"> -->
-    <!-- <origin xyz="0 0 0.05000000000000001" /> -->
-  <!-- </xacro:lidar_v0> -->
-  <!-- <xacro:lidar_gazebo_v0 prefix="top" min_rad="-3.14" max_rad="3.14" min_range="0.02" max_range="10" /> -->
+  <xacro:lidar_v0 prefix="top" parent="base_link">
+    <origin xyz="0 -0.19 0.315" />
+  </xacro:lidar_v0>
+  <xacro:lidar_gazebo_v0 prefix="top" min_rad="-3.14" max_rad="3.14" min_range="0.02" max_range="10" />
   <!-- imu sensor -->
-  <!-- <xacro:imu_v0 prefix="top" parent="base_link"> -->
-    <!-- <origin xyz="0 0 0.05000000000000001" /> -->
-  <!-- </xacro:imu_v0> -->
-  <!-- <xacro:imu_gazebo_v0 prefix="top" /> -->
+  <xacro:imu_v0 prefix="top" parent="base_link">
+    <origin xyz="0 0 0.17" />
+  </xacro:imu_v0>
+  <xacro:imu_gazebo_v0 prefix="top" />
   <xacro:if value="$(arg use_ros2_control)">
     <xacro:include filename="$(find walkie_description)/urdf/walkie/ros2_control.xacro"/>

File: urdf/walkie/imu/imu.gz.xacro (robot description, xacro)
@@ -5,6 +5,6 @@
 			<sensor name="imu_sensor" type="imu">
 				<always_on>1</always_on>
-				<update_rate>40</update_rate>
-				<visualize>false</visualize>
+				<update_rate>50</update_rate>
+				<visualize>true</visualize>
 				<topic>imu</topic>
 			</sensor>

File: urdf/walkie/imu/imu_gz.urdf.xacro (robot description, xacro)
@@ -1,5 +1,5 @@
 <?xml version="1.0"?>
 <robot xmlns:xacro="http://ros.org/wiki/xacro">
-  <xacro:include filename="$(find armmy_omnibot)/urdf/imu/imu.gz.xacro" />
+  <xacro:include filename="$(find walkie_description)/urdf/walkie/imu/imu.gz.xacro" />
   <xacro:macro name="imu_v0" params="prefix parent *joint_origin">
     <joint name="${prefix}_imu_joint" type="fixed">

File: urdf/walkie/lidar/lidar_gz.urdf.xacro (robot description, xacro)
@@ -1,5 +1,5 @@
 <?xml version="1.0"?>
 <robot xmlns:xacro="http://ros.org/wiki/xacro">
-  <xacro:include filename="$(find armmy_omnibot)/urdf/lidar/lidar.gz.xacro" />
+  <xacro:include filename="$(find walkie_description)/urdf/walkie/lidar/lidar.gz.xacro" />
   <xacro:macro name="lidar_v0" params="prefix parent *joint_origin">
     <joint name="${prefix}_lidar_joint" type="fixed">

Commit message: add depth camera

File: robots/gz_walkie.urdf.xacro (robot description, xacro)
@@ -8,4 +8,5 @@
   <xacro:include filename="$(find walkie_description)/urdf/walkie/lidar/lidar_gz.urdf.xacro"/>
   <xacro:include filename="$(find walkie_description)/urdf/walkie/imu/imu_gz.urdf.xacro"/>
+  <xacro:include filename="$(find walkie_description)/urdf/walkie/depth_camera/d415.urdf.xacro"/>
   <!-- =============== Link & Joint =============== -->
   <!-- Base -->
@@ -41,4 +42,9 @@
   </xacro:lidar_v0>
   <xacro:lidar_gazebo_v0 prefix="top" min_rad="-3.14" max_rad="3.14" min_range="0.02" max_range="10" />
+  <!-- depth cam sensor -->
+  <xacro:sensor_d415 name="bottom" parent="base_link" flag_color="1" flag_ir="0" flag_depth="1" updaterate="2">
+    <!-- <origin xyz="0 -0.23813 0.18161" rpy="0 0 -${M_PI/4}"/> -->
+    <origin xyz="0 -0.23813 0.18161" rpy="0 -0.5564807787058716 -${M_PI/2}"/>
+  </xacro:sensor_d415>
   <!-- imu sensor -->
   <xacro:imu_v0 prefix="top" parent="base_link">

File: urdf/walkie/base/base.urdf.xacro (robot description, xacro)
@@ -5,5 +5,5 @@
   <xacro:property name="bass_thickness" value="0.008" />
   <xacro:property name="base_radian" value="0.040" />
-  <xacro:property name="base_mass" value="2.2" />
+  <xacro:property name="base_mass" value="20.2" />
   <xacro:macro name="base_v0" params="parent *joint_origin">
     <joint name="base_link_joint" type="fixed">
