Commit message: add method to change hardware interface via xacro

File: robots/gz_walkie.urdf.xacro (robot description, xacro)
@@ -2,6 +2,5 @@
 <robot name="walkie_bot" xmlns:xacro="http://ros.org/wiki/xacro">
   <xacro:property name="M_PI" value="3.14159274" />
-  <xacro:arg name="use_ros2_control" default="true" />
-  <xacro:arg name="sim_mode" default="true" />
+  <xacro:arg name="ros2_control" default="gazebo" />
   <xacro:include filename="$(find walkie_description)/urdf/walkie/base/base.urdf.xacro"/>
   <xacro:include filename="$(find walkie_description)/urdf/walkie/omni_wheel/gz_omni_wheel.urdf.xacro"/>
@@ -52,6 +51,4 @@
   </xacro:imu_v0>
   <xacro:imu_gazebo_v0 prefix="top" />
-  <xacro:if value="$(arg use_ros2_control)">
-    <xacro:include filename="$(find walkie_description)/urdf/walkie/ros2_control.xacro"/>
-  </xacro:if>
+  <xacro:include filename="$(find walkie_description)/urdf/walkie/ros2_control.xacro" />
 </robot>

File: urdf/walkie/ros2_control.xacro (robot description, xacro)
@@ -1,54 +1,93 @@
 <?xml version="1.0"?>
 <robot xmlns:xacro="http://www.ros.org/wiki/xacro">
-    <xacro:if value="$(arg sim_mode)">
-        <ros2_control name="GazeboSimSystem" type="system">
-          <hardware>
-            <plugin>gz_ros2_control/GazeboSimSystem</plugin>
-          </hardware>
-          <joint name="fl_wheel_joint">
-            <command_interface name="velocity">
-              <param name="min"> -3.14</param>
-              <param name="max"> 3.14</param>
-            </command_interface>
-            <state_interface name="velocity" />
-            <state_interface name="position" />
-          </joint>
-          <joint name="fr_wheel_joint">
-            <command_interface name="velocity">
-              <param name="min"> -3.14</param>
-              <param name="max"> 3.14</param>
-            </command_interface>
-            <state_interface name="velocity" />
-            <state_interface name="position" />
-          </joint>
-          <joint name="bl_wheel_joint">
-            <command_interface name="velocity">
-              <param name="min"> -3.14</param>
-              <param name="max"> 3.14</param>
-            </command_interface>
-            <state_interface name="velocity" />
-            <state_interface name="position" />
-          </joint>
-          <joint name="br_wheel_joint">
-            <command_interface name="velocity">
-              <param name="min"> -3.14</param>
-              <param name="max"> 3.14</param>
-            </command_interface>
-            <state_interface name="velocity" />
-            <state_interface name="position" />
-          </joint>
+  <xacro:macro name="ros2_control" params="ros2_control">
+    <xacro:if value="${ros2_control == 'gazebo'}">
+      <ros2_control name="GazeboSimSystem" type="system">
+        <hardware>
+          <plugin>gz_ros2_control/GazeboSimSystem</plugin>
+        </hardware>
+        <joint name="fl_wheel_joint">
+          <command_interface name="velocity">
+            <param name="min"> -3.14</param>
+            <param name="max"> 3.14</param>
+          </command_interface>
+          <state_interface name="velocity" />
+          <state_interface name="position" />
+        </joint>
+        <joint name="fr_wheel_joint">
+          <command_interface name="velocity">
+            <param name="min"> -3.14</param>
+            <param name="max"> 3.14</param>
+          </command_interface>
+          <state_interface name="velocity" />
+          <state_interface name="position" />
+        </joint>
+        <joint name="br_wheel_joint">
+          <command_interface name="velocity">
+            <param name="min"> -3.14</param>
+            <param name="max"> 3.14</param>
+          </command_interface>
+          <state_interface name="velocity" />
+          <state_interface name="position" />
+        </joint>
+        <joint name="bl_wheel_joint">
+          <command_interface name="velocity">
+            <param name="min"> -3.14</param>
+            <param name="max"> 3.14</param>
+          </command_interface>
+          <state_interface name="velocity" />
+          <state_interface name="position" />
+        </joint>
+      </ros2_control>
+    </xacro:if>
+    <xacro:if value="${ros2_control == 'topic_base'}">
+      <ros2_control name="topic_base_controller" type="system">
+        <hardware>
+          <plugin>topic_based_ros2_control/TopicBasedSystem</plugin>
+          <param name="joint_commands_topic">/drivebase_joint_cmd</param>
+          <param name="joint_states_topic">/drivebase_joint_states</param>
+          <!-- <param name="sum_wrapped_joint_states">true</param> -->
+          <param name="trigger_joint_command_threshold">-1.0</param>
+        </hardware>
+        <joint name="fl_wheel_joint">
+          <command_interface name="velocity">
+            <param name="min"> -16.00</param>
+            <param name="max"> 16.00</param>
+          </command_interface>
+          <state_interface name="velocity" />
+          <state_interface name="position" />
+        </joint>
+        <joint name="fr_wheel_joint">
+          <command_interface name="velocity">
+            <param name="min"> -16.00</param>
+            <param name="max"> 16.00</param>
+          </command_interface>
+          <state_interface name="velocity" />
+          <state_interface name="position" />
+        </joint>
+        <joint name="br_wheel_joint">
+          <command_interface name="velocity">
+            <param name="min"> -16.00</param>
+            <param name="max"> 16.00</param>
+          </command_interface>
+          <state_interface name="velocity" />
+          <state_interface name="position" />
+        </joint>
+        <joint name="bl_wheel_joint">
+          <command_interface name="velocity">
+            <param name="min"> -16.00</param>
+            <param name="max"> 16.00</param>
+          </command_interface>
+          <state_interface name="velocity" />
+          <state_interface name="position" />
+        </joint>
       </ros2_control>
     </xacro:if>
     <gazebo>
-        <plugin name="gz_ros2_control::GazeboSimROS2ControlPlugin" filename="libgz_ros2_control-system.so">
-          <parameters>$(find walkie_description)/config/ros2_controller/my_controllers.yaml</parameters>
-        </plugin>
-        <!-- <plugin filename="libignition-gazebo6-pose-publisher-system.so" name="ignition::gazebo::systems::PosePublisher"> -->
-          <!-- <publish_model_pose>true</publish_model_pose> -->
-          <!-- <publish_link_pose>false</publish_link_pose> -->
-          <!-- <publish_nested_model_pose>true</publish_nested_model_pose> -->
-          <!-- <static_publisher>true</static_publisher> -->
-          <!-- <static_update_frequency>10</static_update_frequency> -->
-        <!-- </plugin> -->
+      <plugin name="gz_ros2_control::GazeboSimROS2ControlPlugin"
+        filename="libgz_ros2_control-system.so">
+        <parameters>$(find walkie_description)/config/ros2_controller/my_controllers.yaml</parameters>
+      </plugin>
     </gazebo>
+  </xacro:macro>
 </robot>

Commit message: fix ros2_control args in robot urdf file

File: robots/gz_walkie.urdf.xacro (robot description, xacro)
@@ -1,6 +1,6 @@
 <?xml version="1.0"?>
-<robot name="walkie_bot" xmlns:xacro="http://ros.org/wiki/xacro">
-  <xacro:property name="M_PI" value="3.14159274" />
-  <xacro:arg name="ros2_control" default="gazebo" />
+<robot xmlns:xacro="http://ros.org/wiki/xacro" name="walkie_bot">
+  <xacro:property name="M_PI" value="3.14159274"/>
+  <xacro:arg name="ros2_control" default="gazebo"/>
   <xacro:include filename="$(find walkie_description)/urdf/walkie/base/base.urdf.xacro"/>
   <xacro:include filename="$(find walkie_description)/urdf/walkie/omni_wheel/gz_omni_wheel.urdf.xacro"/>
@@ -10,35 +10,35 @@
   <!-- =============== Link & Joint =============== -->
   <!-- Base -->
-  <link name="base_footprint" />
+  <link name="base_footprint"/>
   <xacro:base_v0 parent="base_footprint">
-    <origin xyz="0 0 0" rpy="0 0 ${M_PI / 2}" />
+    <origin xyz="0 0 0" rpy="0 0 ${M_PI / 2}"/>
   </xacro:base_v0>
-  <xacro:base_gazebo_v0 />
+  <xacro:base_gazebo_v0/>
   <!-- Wheel -->
   <!-- 1st wheel -->
   <xacro:wheel_v0 prefix="bl" parent="base_link">
-    <origin xyz="0.177622395 0.177622395 0.05" rpy="0 0 -${M_PI/4}" />
-    <axis xyz="0.0 1.0 0.0" />
+    <origin xyz="0.177622395 0.177622395 0.05" rpy="0 0 -${M_PI/4}"/>
+    <axis xyz="0.0 1.0 0.0"/>
   </xacro:wheel_v0>
   <!-- 2nd wheel -->
   <xacro:wheel_v0 prefix="br" parent="base_link">
-    <origin xyz="-0.177622395 0.177622395 0.05" rpy="0 0 ${M_PI/4}" />
-    <axis xyz="0.0 1.0 0.0" />
+    <origin xyz="-0.177622395 0.177622395 0.05" rpy="0 0 ${M_PI/4}"/>
+    <axis xyz="0.0 1.0 0.0"/>
   </xacro:wheel_v0>
   <!-- 3rd wheel -->
   <xacro:wheel_v0 prefix="fr" parent="base_link">
-    <origin xyz="-0.177622395 -0.177622395 0.05" rpy="0 0 ${3*M_PI/4}" />
-    <axis xyz="0.0 1.0 0.0" />
+    <origin xyz="-0.177622395 -0.177622395 0.05" rpy="0 0 ${3*M_PI/4}"/>
+    <axis xyz="0.0 1.0 0.0"/>
   </xacro:wheel_v0>
   <!-- 4th wheel -->
   <xacro:wheel_v0 prefix="fl" parent="base_link">
-    <origin xyz="0.177622395 -0.177622395 0.05" rpy="0 0 ${5*M_PI/4}" />
-    <axis xyz="0.0 1.0 0.0" />
+    <origin xyz="0.177622395 -0.177622395 0.05" rpy="0 0 ${5*M_PI/4}"/>
+    <axis xyz="0.0 1.0 0.0"/>
   </xacro:wheel_v0>
   <!-- lidar sensor -->
   <xacro:lidar_v0 prefix="top" parent="base_link">
-    <origin xyz="0 -0.19 0.315" />
+    <origin xyz="0 -0.19 0.315"/>
   </xacro:lidar_v0>
-  <xacro:lidar_gazebo_v0 prefix="top" min_rad="-3.14" max_rad="3.14" min_range="0.02" max_range="10" />
+  <xacro:lidar_gazebo_v0 prefix="top" min_rad="-3.14" max_rad="3.14" min_range="0.02" max_range="10"/>
   <!-- depth cam sensor -->
   <xacro:sensor_d415 name="bottom" parent="base_link" flag_color="1" flag_ir="0" flag_depth="1" updaterate="2">
@@ -48,7 +48,8 @@
   <!-- imu sensor -->
   <xacro:imu_v0 prefix="top" parent="base_link">
-    <origin xyz="0 0 0.17" />
+    <origin xyz="0 0 0.17"/>
   </xacro:imu_v0>
-  <xacro:imu_gazebo_v0 prefix="top" />
-  <xacro:include filename="$(find walkie_description)/urdf/walkie/ros2_control.xacro" />
+  <xacro:imu_gazebo_v0 prefix="top"/>
+  <xacro:include filename="$(find walkie_description)/urdf/walkie/ros2_control.xacro"/>
+  <xacro:ros2_control ros2_control="$(arg ros2_control)"/>
 </robot>
